Commit message: updated urdf + align/docking nodes + nav2 params updated

File: src/morosai_description/urdf/morosai_agv.urdf.xacro (robot description, xacro)
@@ -1,5 +1,5 @@
 <?xml version="1.0"?>
 <robot xmlns:xacro="http://www.ros.org/wiki/xacro" name="morosai_agv">
-    <xacro_arg name="is_ignition" default="true" />
+    <xacro:arg name="is_ignition" default="true" />
     <!-- Include Gazebo parameters -->
     <xacro:include filename="$(find morosai_description)/urdf/morosai_agv_gazebo.xacro"/>
@@ -7,34 +7,37 @@
     <xacro:include filename="$(find morosai_description)/urdf/morosai_agv_ros2_control.xacro"/>
     <!-- Definizione delle dimensioni principali -->
-    <xacro:property name="base_length" value="0.500"/>  <!-- Lunghezza 500 mm -->
-    <xacro:property name="base_width" value="0.390"/>   <!-- Larghezza 390 mm -->
-    <xacro:property name="wheel_radius" value="0.05"/>  <!-- Raggio stimato della ruota -->
+    <xacro:property name="base_length" value="1.312"/>  <!-- Lunghezza 1312 mm X -->
+    <xacro:property name="base_width" value="1.165"/>   <!-- Larghezza 1165 mm Y -->
+    <xacro:property name="wheel_radius" value="0.05"/>   <!-- Raggio stimato della ruota -->
+    <!-- Definizione parametri posizionamento ruote dai disegni CAD -->
+    <xacro:property name="wheel_x_pos" value="0.435"/>   <!-- Offset X dal centro -->
+    <xacro:property name="wheel_y_pos" value="0.4495"/>  <!-- Offset Y dal centro (899/2) -->
+    <xacro:property name="wheel_z_pos" value="0.05"/>    <!-- Altezza asse Z -->
     <link name="base_footprint"/>
-    <!-- BASE LINK: parallelepipedo -->
     <link name="base_link">
-        <inertial>
-            <origin xyz="0 0 0.11" rpy="0 0 0"/>
-            <mass value="27.508"/>
-            <inertia
-                ixx="4.2886"
-                ixy="-0.010736"
-                ixz="0.0051891"
-                iyy="8.2711"
-                iyz="-0.00085023"
-                izz="4.2714"/>
-        </inertial>
-        <visual>
-            <origin rpy="0 0 0" xyz="0 0 0.11"/>
-            <geometry>
-                <box size="0.5 0.39 0.22"/>
+         <inertial>
+            <origin xyz="0 0 0" rpy="0 0 0"/>
+            <mass value="265.0"/>
+            <inertia
+            ixx="41.3"
+            ixy="-0.1034"
+            ixz="0.04995"
+            iyy="79.7"
+            iyz="-0.0082"
+            izz="41.1"/>
+        </inertial>
+        <visual>
+            <origin rpy="0 0 3.14159" xyz="0 0 0"/>
+            <geometry>
+                <mesh filename="package://morosai_description/meshes/base_link.STL" />
             </geometry>
             <material name="blue">
-                <color rgba="0.0 0.2 1.0 1.0"/>
-            </material>
-        </visual>
-        <collision>
-            <origin rpy="0 0 0" xyz="0 0 0.11"/>
-            <geometry>
-                <box size="0.5 0.39 0.22"/>
+                <color rgba="0.79216 0.81961 0.93333 1" />
+            </material>
+        </visual>
+        <collision>
+            <origin rpy= "0 0 0" xyz="0 0 0"/>
+            <geometry>
+                <mesh filename="package://morosai_description/meshes/agv_morosai-Light1_Telaio-Low.stl" />
             </geometry>
         </collision>
@@ -60,8 +63,8 @@
         <parent link="base_link"/>
         <child link="tof_link"/>
-        <!-- CONFIG CNR STIIMA UPSIDE DOWN -->
-        <!-- <origin xyz="0.25 0 0.186" rpy="0 -1.5708 3.14159"/> -->
-         <!-- INGEL CONFIG MINI AV  -->
-        <origin xyz="0.25 0 0.186" rpy="0 1.5708 0"/>
+        <!-- INGEL CONFIG MINI AV  -->
+        <!-- <origin xyz="0.25 0 0.186" rpy="0 1.5708 0"/> -->
+        <!-- INGEL CONFIG BIG AGV  -->
+        <origin xyz="0.5825 0 0.186" rpy="0 -1.5708 3.14159"/>
     </joint>
     <link name="tof_optical_frame"/>
@@ -69,56 +72,62 @@
         <parent link="tof_link"/>
         <child link="tof_optical_frame"/>
-        <!-- <origin xyz="0 0 0" rpy="0 0 3.14159"/> -->
         <origin xyz="0 0 0" rpy="0 0 1.5708"/>
     </joint>
     <!-- ==== LIDAR FRONT ==== -->
     <link name="lidar_front_link">
-    <visual>
-        <origin xyz="0 0 0" rpy="0 0 0"/>
-        <geometry>
-        <cylinder radius="0.0375" length="0.04"/>
-        </geometry>
-        <material name="red">
-        <color rgba="1.0 0.0 0.0 1.0"/>
-        </material>
-    </visual>
-    </link>
-    <!--
-    Diametralmente opposto significa che il rear avrà x,y con segno opposto.
-    Qui front è a ( +0.2731, +0.306, +0.260 ) e yaw = pi (3.14159),
-    come nel tuo esempio.
-    -->
+        <visual>
+            <origin xyz="0 0 0" rpy="0 0 0"/>
+            <geometry>
+            <cylinder radius="0.0375" length="0.04"/>
+            </geometry>
+            <material name="red">
+            <color rgba="1.0 0.0 0.0 1.0"/>
+            </material>
+        </visual>
+    </link>
     <joint name="lidar_front_joint" type="fixed">
-    <parent link="base_link"/>
-    <child link="lidar_front_link"/>
-    <!-- <origin xyz="0.2731 0.306 0.260" rpy="0 0 3.14159"/> -->
-    <origin xyz="0.2931 0.246 0.260" rpy="0 0 3.14159"/>  <!-- configurazione MINI AGV -->
+        <parent link="base_link"/>
+        <child link="lidar_front_link"/>
+        <!-- configurazione MINI AGV -->
+        <!-- <origin xyz="0.2931 0.246 0.260" rpy="0 0 3.14159"/>   -->
+        <origin xyz="0.608 0.545 0.065" rpy="0 0 3.14159"/>
     </joint>
     <!-- ==== LIDAR REAR ==== -->
     <link name="lidar_rear_link">
-    <visual>
-        <origin xyz="0 0 0" rpy="0 0 0"/>
-        <geometry>
-        <cylinder radius="0.0375" length="0.04"/>
-        </geometry>
-        <material name="red"/>
-    </visual>
-    </link>
-    <!--
-    Rear diametralmente opposto: (-0.2731, -0.306, 0.260)
-    Per “guardare” verso il retro, metti yaw = 0 (in contrapposizione al front che hai ruotato di pi)
-    Nota: per un 2D lidar la rotazione attorno a z non influisce sullo scan, ma è bene essere coerenti.
-    -->
+        <visual>
+            <origin xyz="0 0 0" rpy="0 0 0"/>
+            <geometry>
+            <cylinder radius="0.0375" length="0.04"/>
+            </geometry>
+            <material name="red"/>
+        </visual>
+    </link>
     <joint name="lidar_rear_joint" type="fixed">
-    <parent link="base_link"/>
-    <child link="lidar_rear_link"/>
-    <origin xyz="-0.2731 -0.306 0.260" rpy="0 0 0"/>
-    </joint>
-    <!-- <joint name="lidar_rear_joint" type="fixed">
-        <parent link="base_link"/>
-        <child  link="lidar_rear_link"/>
-        <origin xyz="1.1565 1.0137 0.260" rpy="0 0 -0.03104"/>
-    </joint> -->
+        <parent link="base_link"/>
+        <child link="lidar_rear_link"/>
+        <!-- <origin xyz="-0.2731 -0.306 0.260" rpy="0 0 0"/> -->
+        <origin xyz="-0.608 -0.545 0.065" rpy="0 0 0"/>
+    </joint>
+    <!-- ========================================== -->
+    <!-- OPTICAL HEAD (PGV100 Reader)               -->
+    <!-- ========================================== -->
+    <link name="optical_head_link">
+        <visual>
+            <origin xyz="0 0 0" rpy="0 0 0"/>
+            <geometry>
+                <box size="0.06808 0.06808 0.04998"/>
+            </geometry>
+            <material name="orange">
+                <color rgba="1.0 0.5 0.0 1.0"/>
+            </material>
+        </visual>
+    </link>
+    <joint name="optical_head_joint" type="fixed">
+        <parent link="base_link"/>
+        <child link="optical_head_link"/>
+        <origin xyz="0.475 0.0 0.088" rpy="3.14159265359 0 0"/>
+    </joint>
     <!-- WHEELS -->
+    <!-- FRONT RIGHT -->
     <link name="wheel_front_right">
         <inertial>
@@ -126,10 +135,10 @@
             <mass value="2.91"/>
             <inertia
-                ixx="0.00458012929964188"
-                ixy="-8.16206171695503E-07"
-                ixz="0.000741678448097534"
-                iyy="0.00561604136708303"
-                iyz="3.96551218314105E-06"
-                izz="0.00479467479360652"/>
+            ixx="0.00458012929964188"
+            ixy="-8.16206171695503E-07"
+            ixz="0.000741678448097534"
+            iyy="0.00561604136708303"
+            iyz="3.96551218314105E-06"
+            izz="0.00479467479360652"/>
         </inertial>
         <visual>
@@ -150,10 +159,16 @@
     </link>
     <joint name="wheel_front_right_joint" type="fixed">
-    <!-- CHECK perchè continous non si muove su rviz -->
         <parent link="base_link"/>
         <child link="wheel_front_right"/>
-        <origin rpy="0 0 0" xyz="0.25 -0.195 0.05"/>
-        <axis xyz="0 1 0"/>
-    </joint>
+        <origin rpy="0 0 0" xyz="${wheel_x_pos} ${-wheel_y_pos} ${wheel_z_pos}"/>
+        <axis xyz="0 1 0"/>
+    </joint>
+    <gazebo reference="wheel_front_right">
+        <mu1>100.0</mu1>
+        <mu2>100.0</mu2>
+        <kp>10000000.0</kp>
+        <kd>1.0</kd>
+    </gazebo>
+    <!-- FRONT LEFT -->
     <link name="wheel_front_left">
         <inertial>
@@ -161,10 +176,10 @@
             <mass value="2.91"/>
             <inertia
-                ixx="0.0045801"
-                ixy="8.1621E-07"
-                ixz="-0.00074168"
-                iyy="0.005616"
-                iyz="3.9655E-06"
-                izz="0.0047947" />
+            ixx="0.0045801"
+            ixy="8.1621E-07"
+            ixz="-0.00074168"
+            iyy="0.005616"
+            iyz="3.9655E-06"
+            izz="0.0047947" />
         </inertial>
         <visual>
@@ -187,7 +202,14 @@
         <parent link="base_link"/>
         <child link="wheel_front_left"/>
-        <origin rpy="0 0 0" xyz="0.25 0.195 0.05"/>
-        <axis xyz="0 1 0"/>
-    </joint>
+        <origin rpy="0 0 0" xyz="${wheel_x_pos} ${wheel_y_pos} ${wheel_z_pos}"/>
+        <axis xyz="0 1 0"/>
+    </joint>
+    <gazebo reference="wheel_front_left">
+        <mu1>100.0</mu1>
+        <mu2>100.0</mu2>
+        <kp>10000000.0</kp>
+        <kd>1.0</kd>
+    </gazebo>
+    <!-- REAR RIGHT -->
     <link name="wheel_rear_right">
         <inertial>
@@ -195,10 +217,10 @@
             <mass value="2.91"/>
             <inertia
-                ixx="0.00458012929965282"
-                ixy="-8.16206173013403E-07"
-                ixz="0.00074167844810129"
-                iyy="0.00561604136709717"
-                iyz="3.96551218697627E-06"
-                izz="0.00479467479361136" />
+            ixx="0.00458012929965282"
+            ixy="-8.16206173013403E-07"
+            ixz="0.00074167844810129"
+            iyy="0.00561604136709717"
+            iyz="3.96551218697627E-06"
+            izz="0.00479467479361136" />
         </inertial>
         <visual>
@@ -221,7 +243,14 @@
         <parent link="base_link"/>
         <child link="wheel_rear_right"/>
-        <origin rpy="0 0 0" xyz="-0.25 -0.195 0.05"/>
-        <axis xyz="0 1 0"/>
-    </joint>
+        <origin rpy="0 0 0" xyz="-${wheel_x_pos} -${wheel_y_pos} ${wheel_z_pos}"/>
+        <axis xyz="0 1 0"/>
+    </joint>
+    <gazebo reference="wheel_rear_right">
+        <mu1>100.0</mu1>
+        <mu2>100.0</mu2>
+        <kp>10000000.0</kp>
+        <kd>1.0</kd>
+    </gazebo>
+    <!-- REAR LEFT -->
     <link name="wheel_rear_left">
         <inertial>
@@ -229,10 +258,10 @@
             <mass value="2.91"/>
             <inertia
-                ixx="0.00458012929965168"
-                ixy="8.16206173575887E-07"
-                ixz="-0.000741678448102401"
-                iyy="0.00561604136709495"
-                iyz="3.96551218641184E-06"
-                izz="0.00479467479361022" />
+            ixx="0.00458012929965168"
+            ixy="8.16206173575887E-07"
+            ixz="-0.000741678448102401"
+            iyy="0.00561604136709495"
+            iyz="3.96551218641184E-06"
+            izz="0.00479467479361022" />
         </inertial>
         <visual>
@@ -255,6 +284,12 @@
         <parent link="base_link"/>
         <child link="wheel_rear_left"/>
-        <origin rpy="0 0 0" xyz="-0.25 0.195 0.05"/>
-        <axis xyz="0 1 0"/>
-    </joint>
+        <origin rpy="0 0 0" xyz="-${wheel_x_pos} ${wheel_y_pos} ${wheel_z_pos}"/>
+        <axis xyz="0 1 0"/>
+    </joint>
+    <gazebo reference="wheel_rear_left">
+        <mu1>100.0</mu1>
+        <mu2>100.0</mu2>
+        <kp>10000000.0</kp>
+        <kd>1.0</kd>
+    </gazebo>
 </robot>

Commit message: updated config for AGV final

File: src/morosai_description/urdf/morosai_agv.urdf.xacro (robot description, xacro)
@@ -66,5 +66,5 @@
         <!-- <origin xyz="0.25 0 0.186" rpy="0 1.5708 0"/> -->
         <!-- INGEL CONFIG BIG AGV  -->
-        <origin xyz="0.5825 0 0.186" rpy="0 -1.5708 3.14159"/>
+        <origin xyz="0.5825 0 0.258" rpy="0 -1.5708 3.14159"/>
     </joint>
     <link name="tof_optical_frame"/>
@@ -91,5 +91,5 @@
         <!-- configurazione MINI AGV -->
         <!-- <origin xyz="0.2931 0.246 0.260" rpy="0 0 3.14159"/>   -->
-        <origin xyz="0.608 0.545 0.065" rpy="0 0 3.14159"/>
+        <origin xyz="0.540 0.637 0.098" rpy="0 0 3.14159"/>
     </joint>
     <!-- ==== LIDAR REAR ==== -->
@@ -107,5 +107,6 @@
         <child link="lidar_rear_link"/>
         <!-- <origin xyz="-0.2731 -0.306 0.260" rpy="0 0 0"/> -->
-        <origin xyz="-0.608 -0.545 0.065" rpy="0 0 0"/>
+        <!-- <origin xyz="-0.608 -0.545 0.065" rpy="0 0 0"/> -->
+        <origin xyz="-0.540 -0.637 0.098" rpy="0 0 0"/>
     </joint>
     <!-- ========================================== -->

Commit message: updated params at Ingel for final config

File: src/morosai_description/urdf/morosai_agv.urdf.xacro (robot description, xacro)
@@ -7,10 +7,10 @@
     <xacro:include filename="$(find morosai_description)/urdf/morosai_agv_ros2_control.xacro"/>
     <!-- Definizione delle dimensioni principali -->
-    <xacro:property name="base_length" value="1.312"/>  <!-- Lunghezza 1312 mm X -->
-    <xacro:property name="base_width" value="1.165"/>   <!-- Larghezza 1165 mm Y -->
-    <xacro:property name="wheel_radius" value="0.05"/>   <!-- Raggio stimato della ruota -->
+    <xacro:property name="base_length" value="1.350"/>  <!-- Lunghezza 1312 mm X -->
+    <xacro:property name="base_width" value="1.155"/>   <!-- Larghezza 1165 mm Y -->
+    <xacro:property name="wheel_radius" value="0.081"/>   <!-- Raggio stimato della ruota -->
     <!-- Definizione parametri posizionamento ruote dai disegni CAD -->
-    <xacro:property name="wheel_x_pos" value="0.435"/>   <!-- Offset X dal centro -->
-    <xacro:property name="wheel_y_pos" value="0.4495"/>  <!-- Offset Y dal centro (899/2) -->
+    <xacro:property name="wheel_x_pos" value="0.4175"/>   <!-- Offset X dal centro -->
+    <xacro:property name="wheel_y_pos" value="0.4425"/>  <!-- Offset Y dal centro (899/2) -->
     <xacro:property name="wheel_z_pos" value="0.05"/>    <!-- Altezza asse Z -->
     <link name="base_footprint"/>
@@ -66,5 +66,6 @@
         <!-- <origin xyz="0.25 0 0.186" rpy="0 1.5708 0"/> -->
         <!-- INGEL CONFIG BIG AGV  -->
-        <origin xyz="0.5825 0 0.258" rpy="0 -1.5708 3.14159"/>
+        <!-- <origin xyz="0.5575 0 0.258" rpy="0 -1.5708 3.14159"/> -->
+        <origin xyz="0.5575 0 0.2" rpy="0 -1.5708 3.14159"/>
     </joint>
     <link name="tof_optical_frame"/>
@@ -127,5 +128,5 @@
         <parent link="base_link"/>
         <child link="optical_head_link"/>
-        <origin xyz="0.475 0.0 0.088" rpy="3.14159265359 0 0"/>
+        <origin xyz="0.4375 0.0 0.125" rpy="3.14159265359 0 0"/>
     </joint>
     <!-- WHEELS -->

Commit message: updated map fema, filter pointcloud tof node, watchdog sllidar

File: src/morosai_description/urdf/morosai_agv.urdf.xacro (robot description, xacro)
@@ -67,5 +67,6 @@
         <!-- INGEL CONFIG BIG AGV  -->
         <!-- <origin xyz="0.5575 0 0.258" rpy="0 -1.5708 3.14159"/> -->
-        <origin xyz="0.5575 0 0.2" rpy="0 -1.5708 3.14159"/>
+        <origin xyz="0.5575 0 0.15" rpy="0 -1.57 3.14159"/>
+        <!-- <origin xyz="0.5575 0 0.15" rpy="0 -1.70 3.14159"/> -->
     </joint>
     <link name="tof_optical_frame"/>
